File: EyeBauble/EyeBauble.kicad_pcb (KiCad board)
At the start: 2 copper layers, 17 parts

Commit message: Dunno what I'm committing but this was the latest rev
Parts:
- removed C101: C, Capacitor_SMD:C_0603_1608Metric
- added J101: Conn_01x01_Female, MountingHole:MountingHole_2.5mm, F.Cu at (80.9, 132.2)
- moved D101 25.4 mm to (80.4, 75.0), turned to -0.163322 degrees
- moved D102 23.9 mm to (80.4, 73.1), turned to -0.152434 degrees
- moved D103 21.8 mm to (80.4, 71.2), turned to -0.141546 degrees
- moved D104 20.7 mm to (80.4, 69.3), turned to -0.130658 degrees
- moved D105 18.6 mm to (80.4, 67.4), turned to -0.11977 degrees
- moved D106 17.5 mm to (80.4, 65.5), turned to -0.108882 degrees
- moved D107 16.4 mm to (80.4, 63.6), turned to -0.0979934 degrees
- moved D108 15.4 mm to (80.4, 61.7), turned to -0.0871053 degrees
- moved D109 14.5 mm to (80.4, 59.8), turned to -0.0762171 degrees
- moved D110 13.4 mm to (80.4, 57.9), turned to -0.0653289 degrees
- moved D111 12.6 mm to (80.4, 56.0), turned to -0.0544408 degrees
- moved D112 12.5 mm to (80.4, 54.1), turned to -0.0435526 degrees
- moved D114 11.7 mm to (80.4, 50.3), turned to -0.0217763 degrees
- moved D115 11.7 mm to (80.4, 48.4), turned to -0.0108882 degrees
- moved D113 11.5 mm to (80.4, 52.2), turned to -0.0326645 degrees
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Connections:
- D101 pad 1: (no net) -> /INPUT
Routing:
- net GND: track 0.00 -> 93.2 mm
- net +5V: track 0.00 -> 91.8 mm
- net /INPUT: track 0.00 -> 54.2 mm
- net Net-(D101-Pad3): track 0.00 -> 1.38 mm
- net Net-(D102-Pad3): track 0.00 -> 1.38 mm
- net Net-(D103-Pad3): track 0.00 -> 1.38 mm
- net Net-(D104-Pad3): track 0.00 -> 1.38 mm
- net Net-(D105-Pad3): track 0.00 -> 1.38 mm
- net Net-(D106-Pad3): track 0.00 -> 1.38 mm
- net Net-(D107-Pad3): track 0.00 -> 1.38 mm
- net Net-(D108-Pad3): track 0.00 -> 1.37 mm
- net Net-(D109-Pad3): track 0.00 -> 1.37 mm
- net Net-(D110-Pad3): track 0.00 -> 1.37 mm
- net Net-(D111-Pad3): track 0.00 -> 1.37 mm
- net Net-(D112-Pad3): track 0.00 -> 1.37 mm
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- added copper zone on F.Cu, net +5V
- added copper zone on F.Cu, net /INPUT
- added copper zone on F.Cu, net GND
Other:
- board outline added: 2.7 x 88.4 mm
- net class Default removed
- board text added: "-i+"
